File: SmartSwitchTotalGenerischPC.kicad_sch (KiCad schematic)
At the start: 12 parts, among them J1 Conn_02x05_Odd_Even, J2 Conn_02x05_Odd_Even, J3 Conn_02x04_Odd_Even, Q1 SS8050, U1 XIAO-ESP32-C6

Commit message: refactor: redesign system, replaced BJT w. optocoupler, new input RST_SW
Parts:
- removed J3: Conn_02x04_Odd_Even, Connector_PinHeader_2.54mm:PinHeader_2x04_P2.54mm_Horizontal, symbol Connector_Generic:Conn_02x04_Odd_Even
- removed Q1: SS8050, Package_TO_SOT_SMD:SOT-23W_Handsoldering, symbol Transistor_BJT:SS8050
- removed R3: 3.3k, Resistor_SMD:R_0805_2012Metric_Pad1.20x1.40mm_HandSolder, symbol Device:R
- added C1: 100n, Capacitor_SMD:C_0805_2012Metric_Pad1.18x1.45mm_HandSolder, symbol Device:C
- added IC1: AQW282SZ, Footprints:SOP254P680X230-8N, symbol AQW282SZ:AQW282SZ
- added J3: Conn_02x06_Odd_Even, Connector_PinSocket_2.54mm:PinSocket_2x06_P2.54mm_Horizontal, symbol Connector_Generic:Conn_02x06_Odd_Even
- added R5, R6: 1k, Resistor_SMD:R_0805_2012Metric_Pad1.20x1.40mm_HandSolder, symbol Device:R
- renumbered R4 to R3, R5 to R4
Connections:
- net +5V: now also C1.1
- net GND: now also C1.2, IC1.2 (K1), IC1.4 (K2), IC1.5 (D1), IC1.7 (D3), J3.11 (Pin_11), J3.12 (Pin_12), J3.3 (Pin_3), J3.4 (Pin_4), J3.7 (Pin_7), J3.8 (Pin_8)
- net PWR_LED+: now also J3.1 (Pin_1), J3.2 (Pin_2)
- net PWR_SW+: now also IC1.8 (D4), J3.5 (Pin_5), J3.6 (Pin_6)
- net GPIO19: now reaches R1.2, R2.1
- net GPIO19: now also U1.9 (GPIO19/D8/SCK); no longer U1.1 (GPIO0/A0/D0)
- net GPIO1: now reaches U1.2 (GPIO1/A1/D1)
- net GPIO1: now also R6.1
- net GPIO17: now reaches R3.1
- net GPIO17: now also U1.8 (GPIO17/D7/RX); no longer U1.3 (GPIO2/A2/D2)
- net at U1.4 (GPIO21/D3): no longer R4.1
- net GPIO16: now reaches U1.7 (GPIO16/D6/TX)
- net GPIO16: now also R4.1
- new net: IC1.1 (A1), R6.2
- new net: IC1.3 (A2), R5.2
- new net GPIO2: R5.1, U1.3 (GPIO2/A2/D2)
- new net RST_SW+: IC1.6 (D2), J3.10 (Pin_10), J3.9 (Pin_9)
- no-connect marks 8 -> 7
Other:
- note added: "Butz sagt Kondensator davor um Stromschwankungen durch den Mikrocontroller (Schalt/Logikprozesse) abzufangen und die Powersupply nicht zu belasten."
- note added: "Power / Reset Control"
- note added: "Status LED"
- note added: "System Monitoring"
- moved on the sheet: D1, D2, R1, R2, R3, R4

Commit message: WIP: revised layout w. specific component positions, replaced 2x6 header with 2x6 pin
Parts:
- J3: footprint Connector_PinSocket_2.54mm:PinSocket_2x06_P2.54mm_Horizontal -> Connector_PinHeader_2.54mm:PinHeader_2x06_P2.54mm_Horizontal
Changed lines of the file:
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@@
 			)
 		)
-		(property "Footprint" "Connector_PinSocket_2.54mm:PinSocket_2x06_P2.54mm_Horizontal"
+		(property "Footprint" "Connector_PinHeader_2.54mm:PinHeader_2x06_P2.54mm_Horizontal"
 			(at 242.57 125.73 0)
 			(hide yes)

Commit message: revised: edge cut, silkscreen, machining points, component placement. addition: pulldown resistors f. optocoupler
Parts:
- added R7, R8: 10k, Resistor_SMD:R_0805_2012Metric_Pad1.20x1.40mm_HandSolder, symbol Device:R
Connections:
- net GND: now also R7.2, R8.2
- net GPIO17: now also R1.2, R2.1; no longer R3.1
- net GPIO19: now also R3.1; no longer R1.2, R2.1
- net PWR_LED+: now also J3.10 (Pin_10), J3.9 (Pin_9); no longer J3.1 (Pin_1), J3.2 (Pin_2)
- net RST_SW+: now also J3.1 (Pin_1), J3.2 (Pin_2); no longer J3.10 (Pin_10), J3.9 (Pin_9)
- net at IC1.1 (A1), R6.2: now also R8.1
- net at IC1.3 (A2), R5.2: now also R7.1
- net GPIO20: now reaches U1.10 (GPIO20/D9/MISO)
- net GPIO20: now also R6.1
- net GPIO18: now reaches U1.11 (GPIO18/D10/MOSI)
- net GPIO18: now also R5.1
- net GPIO1: no longer names the net of U1.2 (GPIO1/A1/D1)
- net GPIO1: no longer R6.1
- net GPIO2: no longer names the net of U1.3 (GPIO2/A2/D2)
- net GPIO2: no longer R5.1
Other:
- note added: "<- Pulldown um während dem Einschaltvorgang des ESP floating pin oder false triggers vorzubeugen"
- moved on the sheet: IC1, R5, R6

Commit message: removed: pulldown resistor from switching circuit
Parts:
- removed R7, R8: 10k, Resistor_SMD:R_0805_2012Metric_Pad1.20x1.40mm_HandSolder, symbol Device:R
Other:
- note removed: "<- Pulldown um während dem Einschaltvorgang des ESP floating pin oder false triggers vorzubeugen"
Changed lines of the file:
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@@
 		)
 	)
-	(text "<- Pulldown um während dem Einschaltvorgang des ESP \nfloating pin oder false triggers vorzubeugen"
-		(exclude_from_sim no)
-		(at 68.072 168.402 0)
-		(effects
-			(font
-				(size 1.27 1.27)
-			)
-		)
-	)
 	(text "passthrough"
 		(exclude_from_sim no)
@@
 	)
 	(junction
-		(at 40.64 172.72)
-		(diameter 0)
-		(color 0 0 0 0)
-	)
-	(junction
 		(at 265.43 133.35)
 		(diameter 0)
@@
 	)
 	(junction
-		(at 34.29 172.72)
-		(diameter 0)
-		(color 0 0 0 0)
-	)
-	(junction
-		(at 34.29 153.67)
-		(diameter 0)
-		(color 0 0 0 0)
-	)
-	(junction
 		(at 69.85 161.29)
 		(diameter 0)
@@
 		(color 0 0 0 0)
 	)
-	(junction
-		(at 25.4 158.75)
-		(diameter 0)
-		(color 0 0 0 0)
-	)
 	(no_connect
 		(at 114.3 93.98)
@@
 	(wire
 		(pts
-			(xy 34.29 172.72) (xy 34.29 171.45)
-		)
-		(stroke
-			(width 0)
-			(type default)
-		)
-	)
-	(wire
-		(pts
 			(xy 34.29 153.67) (xy 43.18 153.67)
 		)
@@
 	(wire
 		(pts
-			(xy 34.29 153.67) (xy 34.29 163.83)
-		)
-		(stroke
-			(width 0)
-			(type default)
-		)
-	)
-	(wire
-		(pts
 			(xy 34.29 73.66) (xy 34.29 76.2)
 		)
@@
 	(wire
 		(pts
-			(xy 25.4 158.75) (xy 25.4 163.83)
-		)
-		(stroke
-			(width 0)
-			(type default)
-		)
-	)
-	(wire
-		(pts
 			(xy 21.59 62.23) (xy 21.59 66.04)
 		)
@@
 	(wire
 		(pts
-			(xy 25.4 172.72) (xy 40.64 172.72)
-		)
-		(stroke
-			(width 0)
-			(type default)
-		)
-	)
-	(wire
-		(pts
 			(xy 69.85 161.29) (xy 69.85 172.72)
 		)
@@
 	(wire
 		(pts
-			(xy 25.4 172.72) (xy 25.4 171.45)
-		)
-		(stroke
-			(width 0)
-			(type default)
-		)
-	)
-	(wire
-		(pts
 			(xy 250.19 85.09) (xy 250.19 50.8)
 		)
@@
 	)
 	(symbol
-		(lib_id "Device:R")
-		(at 25.4 167.64 0)
-		(unit 1)
-		(body_style 1)
-		(exclude_from_sim no)
-		(in_bom yes)
-		(on_board yes)
-		(in_pos_files yes)
-		(dnp no)
-		(fields_autoplaced yes)
-		(property "Reference" "R7"
-			(at 27.94 166.3699 0)
-			(show_name no)
-			(do_not_autoplace no)
-			(effects
-				(font
-					(size 1.27 1.27)
-				)
-				(justify left)
-			)
-		)
-		(property "Value" "10k"
-			(at 27.94 168.9099 0)
-			(show_name no)
-			(do_not_autoplace no)
-			(effects
-				(font
-					(size 1.27 1.27)
-				)
-				(justify left)
-			)
-		)
-		(property "Footprint" "Resistor_SMD:R_0805_2012Metric_Pad1.20x1.40mm_HandSolder"
-			(at 23.622 167.64 90)
-			(hide yes)
-			(show_name no)
-			(do_not_autoplace no)
-			(effects
-				(font
-					(size 1.27 1.27)
-				)
-			)
-		)
-		(property "Datasheet" ""
-			(at 25.4 167.64 0)
-			(hide yes)
-			(show_name no)
-			(do_not_autoplace no)
-			(effects
-				(font
-					(size 1.27 1.27)
-				)
-			)
-		)
-		(property "Description" "Resistor"
-			(at 25.4 167.64 0)
-			(hide yes)
-			(show_name no)
-			(do_not_autoplace no)
-			(effects
-				(font
-					(size 1.27 1.27)
-				)
-			)
-		)
-		(pin "1"
-		)
-		(pin "2"
-		)
-		(instances
-			(project "SmartSwitchTotalGenerischPC"
-				(path "/09b4ba7b-4c32-4e0e-8c52-120a08da829d"
-					(reference "R7")
-					(unit 1)
-				)
-			)
-		)
-	)
-	(symbol
 		(lib_id "power:GND")
 		(at 54.61 172.72 0)
@@
 					(unit 1)
 				)
-			)
-		)
-	)
-	(symbol
-		(lib_id "Device:R")
-		(at 34.29 167.64 0)
-		(unit 1)
-		(body_style 1)
-		(exclude_from_sim no)
-		(in_bom yes)
-		(on_board yes)
-		(in_pos_files yes)
-		(dnp no)
-		(fields_autoplaced yes)
-		(property "Reference" "R8"
-			(at 36.83 166.3699 0)
-			(show_name no)
-			(do_not_autoplace no)
-			(effects
-				(font
-					(size 1.27 1.27)
-				)
-				(justify left)
-			)
-		)
-		(property "Value" "10k"
-			(at 36.83 168.9099 0)
-			(show_name no)
-			(do_not_autoplace no)
-			(effects
-				(font
-					(size 1.27 1.27)
-				)
-				(justify left)
-			)
-		)
-		(property "Footprint" "Resistor_SMD:R_0805_2012Metric_Pad1.20x1.40mm_HandSolder"
-			(at 32.512 167.64 90)
-			(hide yes)
-			(show_name no)
-			(do_not_autoplace no)
-			(effects
-				(font
-					(size 1.27 1.27)
-				)
-			)
-		)
-		(property "Datasheet" ""
-			(at 34.29 167.64 0)
-			(hide yes)
-			(show_name no)
-			(do_not_autoplace no)
-			(effects
-				(font
-					(size 1.27 1.27)
-				)
-			)
-		)
-		(property "Description" "Resistor"
-			(at 34.29 167.64 0)
-			(hide yes)
-			(show_name no)
-			(do_not_autoplace no)
-			(effects
-				(font
-					(size 1.27 1.27)
-				)
-			)
-		)
-		(pin "1"
-		)
-		(pin "2"
-		)
-		(instances
-			(project "SmartSwitchTotalGenerischPC"
-				(path "/09b4ba7b-4c32-4e0e-8c52-120a08da829d"
-					(reference "R8")
-					(unit 1)
-				)
